Commit message: point to new meshes in urdf

File: phosphobot/resources/urdf/ur5e/urdf/ur5e.urdf (robot description, URDF)
Before this commit: robot ur5e, 13 links, 12 joints
Links:
- link base_link_inertia: geometry collision mesh filename=package://ur5e/meshes/base.stl; visual mesh filename=package://ur5e/meshes/base.stl
- link forearm_link: geometry collision mesh filename=package://ur5e/meshes/forearm.stl; visual mesh filename=package://ur5e/meshes/forearm.stl
- link shoulder_link: geometry collision mesh filename=package://ur5e/meshes/shoulder.stl; visual mesh filename=package://ur5e/meshes/shoulder.stl
- link upper_arm_link: geometry collision mesh filename=package://ur5e/meshes/upperarm.stl; visual mesh filename=package://ur5e/meshes/upperarm.stl
- link wrist_1_link: geometry collision mesh filename=package://ur5e/meshes/wrist1.stl; visual mesh filename=package://ur5e/meshes/wrist1.stl
- link wrist_2_link: geometry collision mesh filename=package://ur5e/meshes/wrist2.stl; visual mesh filename=package://ur5e/meshes/wrist2.stl
- link wrist_3_link: geometry collision mesh filename=package://ur5e/meshes/wrist3.stl; visual mesh filename=package://ur5e/meshes/wrist3.stl
